File: _autosave-Keyboard3x3.kicad_sch (KiCad schematic)
At the start: 24 parts, among them SW1 SW_Push, U1 ATmega32U4-A, Y1 16MHz

Commit message: 1/2/2024: Completed wiring
Parts:
- removed D1, D2, D3, D4: D_Small, Diode_SMD:D_SOD-123, symbol Device:D_Small
- removed MX1, MX2, MX3, MX4: MX-NoLED, MX_Alps_Hybrid:MX-1U, symbol MX_Alps_Hybrid:MX-NoLED
- C1: renamed from C7; footprint Capacitor_SMD:C_0805_2012Metric -> (none)
- C2: renamed from C1; footprint Capacitor_SMD:C_0805_2012Metric -> (none)
- C3: renamed from C2; footprint Capacitor_SMD:C_0805_2012Metric -> (none)
- C4: renamed from C3; footprint Capacitor_SMD:C_0805_2012Metric -> (none)
- C5: renamed from C6; footprint Capacitor_SMD:C_0805_2012Metric -> (none)
- C6: renamed from C5; footprint Capacitor_SMD:C_0805_2012Metric -> (none)
- C7: renamed from C4; footprint Capacitor_SMD:C_0805_2012Metric -> (none)
- F1: footprint Fuse:Fuse_1206_3216Metric -> (none)
- R1: renamed from R4; footprint Resistor_SMD:R_0805_2012Metric -> (none)
- R2: footprint Resistor_SMD:R_0805_2012Metric -> (none)
- R3: renamed from R1; footprint Resistor_SMD:R_0805_2012Metric -> (none)
- R4: renamed from R3; footprint Resistor_SMD:R_0805_2012Metric -> (none)
- SW1: footprint random-keyboard-parts:SKQG-1155865 -> (none)
- USB1: footprint random-keyboard-parts:Molex-0548190589 -> (none)
- Y1: footprint Crystal:Crystal_SMD_3225-4Pin_3.2x2.5mm -> (none)
Connections:
- net COL0: no longer names the net of U1.28 (PB4)
- net COL1: no longer names the net of U1.29 (PB5)
- net ROW0: no longer names the net of U1.30 (PB6)
- net ROW1: no longer names the net of U1.27 (PD7)
