File: Keyboard3x3.kicad_pcb (KiCad board)
At the start: 2 copper layers, 67.3 x 38.1 mm, 24 parts, among them SW1 SW_Push, U1 ATmega32U4-A, Y1 16MHz

Commit message: 1/2/2024: Finished and printed
Parts:
- moved D1 2.54 mm to (86.8, 57.2)
- moved D2 2.54 mm to (86.8, 76.3)
- moved D3 2.54 mm to (105.8, 57.2)
- moved D4 2.54 mm to (105.8, 76.3)
- moved MX1 2.54 mm to (78.8, 57.2)
- moved MX2 2.54 mm to (78.8, 76.3)
- moved MX3 2.54 mm to (97.9, 57.2)
- moved MX4 2.54 mm to (97.9, 76.3)
- moved Y1 0.64 mm to (61.4, 55.8)
- moved C4 0.63 mm to (65.2, 55.8)
Routing:
- net COL1: track 49.1 -> 51.6 mm
- net ROW0: track 42.2 -> 44.7 mm
- net COL0: track 29.7 -> 32.3 mm
- net ROW1: track 47.0 -> 48.1 mm
- net Net-(U1-XTAL2): track 9.19 -> 9.82 mm
- net Net-(U1-XTAL1): track 8.15 -> 8.75 mm
- added copper zone on B.Cu, net GND
Other:
- board size 67.3 x 38.1 mm -> 69.8 x 38.1 mm
- board text added: "Nathan Lemma Keyboard 1 3x3"
