File: Keyboard3x3.kicad_sch (KiCad schematic)
At the start: 24 parts, among them SW1 SW_Push, U1 ATmega32U4-A, Y1 16MHz

Commit message: 1/2/2024: Finished and printed
Connections:
- net COL0: now also U1.29 (PB5); no longer U1.28 (PB4)
- net COL1: now also U1.28 (PB4); no longer U1.29 (PB5)
- net ROW0: now also U1.27 (PD7); no longer U1.30 (PB6)
- net ROW1: now also U1.30 (PB6); no longer U1.27 (PD7)
Changed lines of the file:
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@@
     )
   )
-  (global_label "ROW1" (shape input) (at 162.56 99.06 0) (fields_autoplaced)
+  (global_label "ROW0" (shape input) (at 162.56 99.06 0) (fields_autoplaced)
     (effects (font (size 1.27 1.27)) (justify left))
     (property "Intersheetrefs" "${INTERSHEET_REFS}" (at 170.8066 99.06 0)
@@
     )
   )
-  (global_label "COL1" (shape input) (at 162.56 63.5 0) (fields_autoplaced)
+  (global_label "COL0" (shape input) (at 162.56 63.5 0) (fields_autoplaced)
     (effects (font (size 1.27 1.27)) (justify left))
     (property "Intersheetrefs" "${INTERSHEET_REFS}" (at 170.3833 63.5 0)
@@
     )
   )
-  (global_label "COL0" (shape input) (at 162.56 60.96 0) (fields_autoplaced)
+  (global_label "COL1" (shape input) (at 162.56 60.96 0) (fields_autoplaced)
     (effects (font (size 1.27 1.27)) (justify left))
     (property "Intersheetrefs" "${INTERSHEET_REFS}" (at 170.3833 60.96 0)
@@
     )
   )
-  (global_label "ROW0" (shape input) (at 162.56 66.04 0) (fields_autoplaced)
+  (global_label "ROW1" (shape input) (at 162.56 66.04 0) (fields_autoplaced)
     (effects (font (size 1.27 1.27)) (justify left))
     (property "Intersheetrefs" "${INTERSHEET_REFS}" (at 170.8066 66.04 0)
